File: RadioBridge.brd (EAGLE design)
At the start: 34.3 x 57.1 mm, 17 parts, among them IC1 ATMEGA328P_TQFP, IC2 MCP1642B-50I/MS, J1 ICSP, J2 FTDI_HEADER, J3 B2B-XH-A(LF)(SN), Y1 16MHz

Commit message: In progress
Parts:
- removed C2: 22pF, SparkFun-Passives:0603-CAP
- removed C3, C4, C5: (no value), SparkFun-Passives:0805
- removed IC2: MCP1642B-50I/MS, SparkFun-IC-Power:MSOP8
- removed J3: B2B-XH-A(LF)(SN), B2B-XH-A(LF)(SN):SHDR2W64P0X250_1X2_740X575X700
- removed L1: 744042004, SparkFun-Passives:1919(4848_METRIC)
- removed Y1: 16MHz, SparkFun-Clocks:CRYSTAL-SMD-5X3.2-4PAD
- added BT2: LIPO-OUTLINE1100, SparkFun-Batteries:LIPO-1000
- added C8, C9: 10uF, microbuilder:0805
- added CN4: USB, microbuilder:USB-MINIB_LARGER
- added CN5: BATT_IN_JST, microbuilder:JSTPH2
- added JP1, JP9: PWR_IN_0.1, microbuilder:1X02_OVAL
- added LED4: STAT1-ORANGE, microbuilder:CHIPLED_0805
- added LED5: STAT2-GREEN, microbuilder:CHIPLED_0805
- added LED6: Power-RED, microbuilder:CHIPLED_0805
- added R10: 10k, SparkFun-Passives:0603-RES
- added R11: 10K, SparkFun-Passives:0603-RES
- added R6, R8, R9: 150, SparkFun-Passives:0603-RES
- added U2: MCP73833T-AMI/MF, microbuilder:DFN10_3X3MM
- C1: value 22pF -> .1uF; device SparkFun-Passives:0603-CAP -> microbuilder:0805
- moved J2 50.9 mm to (7.11, 54.1)
- moved R1 20.6 mm to (12.7, 8.13), turned to 0 degrees
- moved C1 16.9 mm to (19.1, 11.4), turned to 0 degrees
- moved J1 12.6 mm to (14.0, 5.08), turned to 180 degrees
- moved IC1 10.9 mm to (12.7, 15.2), turned to 135 degrees
- moved S1 8.13 mm to (20.3, 5.08)
- turned D1 to 0 degrees
Connections:
- removed net N$1: C1.2, IC1.7, Y1.3
- removed net N$2: C2.2, IC1.8, Y1.1
- removed net REG_SW: IC2.5, L1.P$1
- removed net REG_VIN: C5.1, IC2.1, IC2.8, J3.1, L1.P$2
- new net +3.3V: C1.1, D1.C, IC1.18, IC1.20, IC1.4, IC1.6, JP1.2, R1.2
- new net 5.0V: C8.1, CN4.VBUS, JP9.2, LED4.A, LED5.A, LED6.A, U2.P$1, U2.P$2
- new net BATT1: C9.1, CN5.2, U2.P$10, U2.P$9
- new net N$13: LED4.C, R6.2
- new net N$14: LED5.C, R8.2
- new net N$15: R6.1, U2.P$3
- new net N$17: R8.1, U2.P$4
- new net N$18: LED6.C, R9.1
- new net N$19: R10.2, U2.P$6
- new net N$20: R9.2, U2.P$7
- new net N$21: R11.2, U2.P$8
- new net VIN: U$1.P$9, U$2.P$1
- net +5V: no longer C3.1, C4.1, D1.C, IC1.18, IC1.20, IC1.4, IC1.6, IC2.4, R1.2, U$1.P$9, U$2.P$1
- net GND: now also C1.2, C8.2, C9.2, CN4.GND, CN5.1, JP1.1, JP9.1, R10.1, R11.1, U2.P$5; no longer C1.1, C2.1, C3.2, C4.2, C5.2, IC2.6, IC2.7, J3.2
Routing:
- net RST: track 69.8 -> 0.00 mm
- net MOSI: track 68.5 -> 0.00 mm, vias 3 -> 0
- net MISO: track 68.2 -> 0.00 mm
- net D5: track 56.4 -> 0.00 mm
- net SCK: track 54.4 -> 0.00 mm, vias 1 -> 0
- net RX: track 44.6 -> 0.00 mm
- net GND: track 41.2 -> 0.00 mm, vias 8 -> 0
- net REG_VIN: track 33.2 -> 0.00 mm, vias 1 -> 0
- net TX: track 30.7 -> 0.00 mm, vias 2 -> 0
- net D8: track 27.4 -> 0.00 mm, vias 1 -> 0
- net D2: track 27.3 -> 0.00 mm
- net +5V: track 19.6 -> 0.00 mm, vias 3 -> 0
- net D7: track 18.8 -> 0.00 mm
- net D3: track 14.6 -> 0.00 mm, vias 2 -> 0
- net D4: track 10.5 -> 0.00 mm
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- added copper zone on layer 1, net BATT1
- removed copper zone on layer 16, net +5V
- removed copper zone on layer 16, net N$3
- removed copper zone on layer 1, net N$4
Other:
- board text added: "+3.3V Reg"
- board text added: "+5V"
- board text removed: "3.3V"

Commit message: Completed V1.0 circuit
Parts:
- removed BT2: LIPO-OUTLINE1100, SparkFun-Batteries:LIPO-1000
- removed C8: 10uF, microbuilder:0805
- removed CN4: USB, microbuilder:USB-MINIB_LARGER
- removed R10: 10k, SparkFun-Passives:0603-RES
- removed R11: 10K, SparkFun-Passives:0603-RES
- removed R9: 150, SparkFun-Passives:0603-RES
- added C2: 10uF, microbuilder:0805
- added CN1: MF-CON-MICROUSB-RIGHT, MF_Connectors:MICROUSB-RIGHT
- added R2, R3: 2.2k, SparkFun-Passives:0603-RES
- added R4, R5: 150, SparkFun-Passives:0603-RES
- added R7: 10k, SparkFun-Passives:0603-RES
- C1: value .1uF -> 0.1uF; device microbuilder:0805 -> SparkFun-Capacitors:0603
- R8: value 150 -> 10K
- moved J2 13.5 mm to (19.6, 48.8), turned to 180 degrees
- moved D1 11.2 mm to (7.87, 19.3), turned to 225 degrees
- moved R8 10.8 mm to (24.6, 19.6), turned to 180 degrees
- moved R6 5.57 mm to (11.7, 24.1), turned to 270 degrees
- moved LED6 4.32 mm to (11.7, 27.9)
- moved LED4 4.20 mm to (14.0, 27.9)
- moved LED5 4.10 mm to (16.3, 27.9)
- moved U$1 2.27 mm to (12.4, 45.2), turned to 180 degrees
- moved C1 1.27 mm to (18.0, 12.2), turned to 45 degrees
- moved S1 0.76 mm to (21.1, 5.08)
- moved IC1 0.51 mm to (12.7, 15.7)
- renumbered C9 to C3, CN5 to CN2, JP9 to JP2, U2 to IC2
Connections:
- new net RXI: J2.3, R2.1
- new net TXO: J2.2, R3.1
- net +3.3V: now also J1.2
- net +5V: no longer J1.2
- net 5.0V: now also C2.1, CN1.1; no longer C8.1, CN4.VBUS
- net GND: now also C2.2, CN1.5, CN1.S1, CN1.S2, CN1.S3, CN1.S4, CN1.S5, CN1.S6, R7.1, R8.1; no longer C8.2, CN4.GND, R10.1, R11.1
- net N$13: now also R5.2; no longer R6.2
- net N$14: now also R4.2; no longer R8.2
- net N$15: now also R5.1; no longer R6.1
- net N$17: now also R4.1; no longer R8.1
- net N$18: now also R6.1; no longer R9.1
- net N$19: now also R7.2; no longer R10.2
- net N$20: now also R6.2; no longer R9.2
- net N$21: now also R8.2; no longer R11.2
- net RX: now also R2.2; no longer J2.3
- net TX: now also R3.2; no longer J2.2
Routing:
- net RST: track 0.00 -> 96.3 mm
- net D2: track 0.00 -> 66.0 mm, vias 0 -> 1
- net SCK: track 0.00 -> 65.6 mm
- net MOSI: track 0.00 -> 65.6 mm, vias 0 -> 1
- net TXO: track 0.00 -> 64.6 mm
- net MISO: track 0.00 -> 63.9 mm, vias 0 -> 2
- net VIN: track 0.00 -> 58.7 mm
- net +3.3V: track 0.00 -> 55.9 mm, vias 0 -> 1
- net D5: track 0.00 -> 51.4 mm, vias 0 -> 1
- net D8: track 0.00 -> 47.2 mm, vias 0 -> 1
- net RXI: track 0.00 -> 46.6 mm
- net 5.0V: track 0.00 -> 40.1 mm, vias 0 -> 2
- net N$20: track 0.00 -> 23.4 mm
- net GND: track 0.00 -> 21.8 mm, vias 0 -> 5
- net D4: track 0.00 -> 20.0 mm, vias 0 -> 2
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- added copper zone on layer 1, net 5.0V
Other:
- board size 34.3 x 57.1 mm -> 31.8 x 58.4 mm
- board text added: "TinkerTech BTLE/900MHz Radio Bridge V1.0 Date: 10-11-17"
- board text removed: "TinkerTech BTLE/900MHz Radio Bridge V1.0 9/29/17"
