File: RadioBridge.sch (EAGLE design)
At the start: 17 parts, among them IC1 ATMEGA328P_TQFP, IC2 MCP1642B-50I/MS, J1 ICSP, J2 FTDI_HEADER, J3 B2B-XH-A(LF)(SN), Y1 16MHz

Commit message: In progress
Parts:
- removed C2: 22pF, SparkFun-Passives:CAP0603-CAP
- removed C3, C4, C5: (no value), SparkFun-Passives:CAP0805
- removed IC2: MCP1642B-50I/MS, SparkFun-IC-Power:MCP1642B-50I/MS
- removed J3: B2B-XH-A(LF)(SN), B2B-XH-A(LF)(SN):B2B-XH-A(LF)(SN)
- removed L1: 744042004, SparkFun-Passives:INDUCTOR
- removed Y1: 16MHz, SparkFun-Clocks:CRYSTAL-16MHZSMD-5X3.2
- added BT2: LIPO-OUTLINE1100, SparkFun-Batteries:LIPO-OUTLINE1100
- added C8, C9: 10uF, microbuilder:CAP_CERAMIC0805
- added CN4: USB, microbuilder:USBMINIBLARGE
- added CN5: BATT_IN_JST, microbuilder:JST_2PIN
- added JP1, JP9: PWR_IN_0.1, microbuilder:HEADER-1X2
- added LED4: STAT1-ORANGE, microbuilder:LED0805
- added LED5: STAT2-GREEN, microbuilder:LED0805
- added LED6: Power-RED, microbuilder:LED0805
- added R10: 10k, SparkFun-Passives:RESISTOR0603-RES
- added R11: 10K, SparkFun-Passives:RESISTOR0603-RES
- added R6, R8, R9: 150, SparkFun-Passives:RESISTOR0603-RES
- added U2: MCP73833T-AMI/MF, microbuilder:MCP73833DFN
- C1: value 22pF -> .1uF; device SparkFun-Passives:CAP0603-CAP -> microbuilder:CAP_CERAMIC0805
Connections:
- removed net N$1: C1.2, IC1.PB6(XTAL1/TOSC1), Y1.2
- removed net N$2: C2.2, IC1.PB7(XTAL2/TOSC2), Y1.1
- removed net REG_SW: IC2.SW, L1.1
- removed net REG_VIN: C5.1, IC2.EN, IC2.VIN, J3.1, L1.2
- new net +3.3V: C1.P$1, D1.C, IC1.AREF, IC1.AVCC, IC1.VCC@4, IC1.VCC@6, JP1.2, R1.2
- new net 5.0V: C8.P$1, CN4.VBUS, JP9.2, LED4.A, LED5.A, LED6.A, U2.VDD1, U2.VDD2
- new net BATT1: C9.P$1, CN5.2, U2.VBAT1, U2.VBAT2
- new net N$13: LED4.C, R6.2
- new net N$14: LED5.C, R8.2
- new net N$15: R6.1, U2.STAT1
- new net N$17: R8.1, U2.STAT2
- new net N$18: LED6.C, R9.1
- new net N$19: R10.2, U2.PROG
- new net N$20: R9.2, U2.PG
- new net N$21: R11.2, U2.THERM
- new net VIN: U$1.VIN, U$2.VIN
- net +5V: no longer C3.1, C4.1, D1.C, IC1.AREF, IC1.AVCC, IC1.VCC@4, IC1.VCC@6, IC2.VOUT, R1.2, U$1.VIN, U$2.VIN
- net GND: now also C1.P$2, C8.P$2, C9.P$2, CN4.GND, CN5.1, JP1.1, JP9.1, R10.1, R11.1, U2.GND; no longer C1.1, C2.1, C3.2, C4.2, C5.2, IC2.PGND, IC2.SGND, J3.2
Other:
- note added: "1.0K = 1000mA"
- note added: "10K = 100mA"
- note added: "10K NTC Thermistor"
- note added: "2.0K = 500mA"
- note added: "5.0K = 200mA"
- note added: "No Thermistor"
- note added: "RT1 = 0 RT2 = NC THERM=10K"
- note added: "RT1 = TBD RT2 = TBD"
- moved on the sheet: C1, D1, IC1, J1, J2, R1, S1

Commit message: Completed V1.0 circuit
Parts:
- removed BT2: LIPO-OUTLINE1100, SparkFun-Batteries:LIPO-OUTLINE1100
- removed CN4: USB, microbuilder:USBMINIBLARGE
- removed R11: 10K, SparkFun-Passives:RESISTOR0603-RES
- removed R9: 150, SparkFun-Passives:RESISTOR0603-RES
- added CN1: MF-CON-MICROUSB-RIGHT, MF_Connectors:USB_MICRO_RIGHT
- added R2, R3: 2.2k, SparkFun-Passives:RESISTOR0603-RES
- added R4, R5: 150, SparkFun-Passives:RESISTOR0603-RES
- C1: value .1uF -> 0.1uF; device microbuilder:CAP_CERAMIC0805 -> SparkFun-Capacitors:0.1UF-0603-25V-(+80/-20%)
- R8: value 150 -> 10K
- renumbered C8 to C2, C9 to C3, CN5 to CN2, JP9 to JP2, R10 to R7, U2 to IC2
Connections:
- new net RXI: J2.RXI, R2.1
- new net TXO: J2.TXO, R3.1
- net +3.3V: now also C1.1, J1.2; no longer C1.P$1
- net +5V: no longer J1.2
- net 5.0V: now also CN1.5V; no longer CN4.VBUS
- net GND: now also C1.2, CN1.GND, CN1.SLD, R8.1; no longer C1.P$2, CN4.GND, R11.1
- net N$13: now also R5.2; no longer R6.2
- net N$14: now also R4.2; no longer R8.2
- net N$15: now also R5.1; no longer R6.1
- net N$17: now also R4.1; no longer R8.1
- net N$18: now also R6.1; no longer R9.1
- net N$20: now also R6.2; no longer R9.2
- net N$21: now also R8.2; no longer R11.2
- net RX: now also R2.2; no longer J2.RXI
- net TX: now also R3.2; no longer J2.TXO
Other:
- moved on the sheet: J2, R6, R8
